File: encoder_driver.kicad_sch (KiCad schematic)
At the start: 21 parts, among them J1 Conn_01x10_Female, J2 Conn_01x10_Female, J3 Conn_01x06, J4 Conn_01x02_Male, Q1 Si2319CDS, U1 AS5045B, U2 AM26LS31CD, U3 AM26LV32xD

Commit message: edit schematic
Connections:
- net +5V: now also R6.2, U3.16 (VDD)
Other:
- moved on the sheet: C1, C2, C3, C4, C5, C6, D1, J1, J2, J3, J4, Q1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

Commit message: lots of layout
Parts:
- R3, R4, R5: footprint Resistor_SMD:R_0402_1005Metric -> Resistor_SMD:R_0603_1608Metric
Connections:
- net +5V: no longer R6.2, U3.16 (VDD)
- net ENC_A: now also J3.5 (Pin_5); no longer J3.4 (Pin_4)
- net ENC_B: now also J3.4 (Pin_4); no longer J3.3 (Pin_3)
- net ENC_C: now also J3.3 (Pin_3); no longer J3.2 (Pin_2)
- net GND: no longer C3.2, J2.10 (Pin_10), J2.8 (Pin_8), J3.6 (Pin_6)
- net TEMP: now also J3.2 (Pin_2); no longer J3.5 (Pin_5)
- net VIN: no longer J2.9 (Pin_9)
- net _GND: now reaches U3.8 (GND)
- net _GND: now also C3.2, J2.10 (Pin_10), J2.8 (Pin_8), J3.6 (Pin_6)
- net V_+5 renamed _+5
- net _+5: now also J2.9 (Pin_9), R6.2, U3.16 (VDD)
Other:
- moved on the sheet: C1, C2

Commit message: edits
Parts:
- J3: footprint Connector_PinHeader_2.54mm:PinHeader_1x06_P2.54mm_Vertical -> Connector_JST:my_JST_1x06_P2.00mm_Vertical
Changed lines of the file:
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@@
       (effects (font (size 1.27 1.27)) (justify left) hide)
     )
-    (property "Footprint" "Connector_PinHeader_2.54mm:PinHeader_1x06_P2.54mm_Vertical" (id 2) (at 239.014 60.96 0)
+    (property "Footprint" "Connector_JST:my_JST_1x06_P2.00mm_Vertical" (id 2) (at 239.014 60.96 0)
       (effects (font (size 1.27 1.27)) hide)
     )
@@
     )
     (path "/ee1d3956-2b26-4116-9888-5d1a66138202"
-      (reference "J3") (unit 1) (value "Conn_01x06") (footprint "Connector_PinHeader_2.54mm:PinHeader_1x06_P2.54mm_Vertical")
+      (reference "J3") (unit 1) (value "Conn_01x06") (footprint "Connector_JST:my_JST_1x06_P2.00mm_Vertical")
     )
     (path "/7d4300d2-37a7-4b79-b1d5-c65e1c7e75ea"
