File: encoder_driver.kicad_sch (KiCad schematic)
At the start: 40 parts, among them J1 Conn_01x08_Female, J2 Conn_01x08_Female, J3 Conn_01x02_Male, J4 Conn_01x07, J5 Conn_01x08_Female, Q1 Si2319CDS, U1 TLE5012b, U2 MCP6L01Rx-xOT, U3 XC6206PxxxMR, U4 B0505T-1W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

Commit message: submitted to jlcpcb
Parts:
- added C4: 4.7uF, Capacitor_SMD:C_0603_1608Metric, symbol Device:C_Small
- C9: value 1uF -> 10uF
- J1, J2, J3, J4, J5, U1: now left out of the parts list
- Q1: LCSC C5122036 -> C558254
Connections:
- net B+5V: now also C4.1
- net BGND: now also C4.2
Other:
- moved on the sheet: C10, C9

Commit message: submitted to jlcpcb
Parts:
- C1, C2: LCSC C14663 -> C346191
- C11, C5, C6, C8: LCSC C14663 -> C361203
- R10, R11, R12, R14: LCSC C25803 -> C269673
- R13, R9: LCSC C23186 -> C103055
- R8: LCSC C25803 -> C14675
Changed lines of the file:
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@@
       (effects (font (size 1.27 1.27)) hide)
     )
-    (property "LCSC" "C25803" (id 4) (at 83.82 165.1 0)
+    (property "LCSC" "C269673" (id 4) (at 83.82 165.1 0)
       (effects (font (size 1.27 1.27)) hide)
     )
@@
       (effects (font (size 1.27 1.27)) hide)
     )
-    (property "LCSC" "C14663" (id 4) (at 146.05 110.49 0)
+    (property "LCSC" "C361203" (id 4) (at 146.05 110.49 0)
       (effects (font (size 1.27 1.27)) hide)
     )
@@
       (effects (font (size 1.27 1.27)) hide)
     )
-    (property "LCSC" "C14663" (id 4) (at 191.77 105.41 0)
+    (property "LCSC" "C346191" (id 4) (at 191.77 105.41 0)
       (effects (font (size 1.27 1.27)) hide)
     )
@@
       (effects (font (size 1.27 1.27)) hide)
     )
-    (property "LCSC" "C14663" (id 4) (at 110.49 118.11 0)
+    (property "LCSC" "C361203" (id 4) (at 110.49 118.11 0)
       (effects (font (size 1.27 1.27)) hide)
     )
@@
       (effects (font (size 1.27 1.27)) hide)
     )
-    (property "LCSC" "C25803" (id 4) (at 68.58 148.59 0)
+    (property "LCSC" "C269673" (id 4) (at 68.58 148.59 0)
       (effects (font (size 1.27 1.27)) hide)
     )
@@
       (effects (font (size 1.27 1.27)) hide)
     )
-    (property "LCSC" "C14663" (id 4) (at 256.54 60.96 0)
+    (property "LCSC" "C346191" (id 4) (at 256.54 60.96 0)
       (effects (font (size 1.27 1.27)) hide)
     )
@@
       (effects (font (size 1.27 1.27)) hide)
     )
-    (property "LCSC" "C14663" (id 4) (at 95.25 118.11 0)
+    (property "LCSC" "C361203" (id 4) (at 95.25 118.11 0)
       (effects (font (size 1.27 1.27)) hide)
     )
@@
       (effects (font (size 1.27 1.27)) hide)
     )
-    (property "LCSC" "C14663" (id 4) (at 162.56 109.22 0)
+    (property "LCSC" "C361203" (id 4) (at 162.56 109.22 0)
       (effects (font (size 1.27 1.27)) hide)
     )
@@
       (effects (font (size 1.27 1.27)) hide)
     )
-    (property "LCSC" "C23186" (id 4) (at 60.96 138.43 0)
+    (property "LCSC" "C103055" (id 4) (at 60.96 138.43 0)
       (effects (font (size 1.27 1.27)) hide)
     )
@@
       (effects (font (size 1.27 1.27)) hide)
     )
-    (property "LCSC" "C25803" (id 4) (at 210.82 113.03 0)
+    (property "LCSC" "C14675" (id 4) (at 210.82 113.03 0)
       (effects (font (size 1.27 1.27)) hide)
     )
@@
       (effects (font (size 1.27 1.27)) hide)
     )
-    (property "LCSC" "C23186" (id 4) (at 60.96 168.91 0)
+    (property "LCSC" "C103055" (id 4) (at 60.96 168.91 0)
       (effects (font (size 1.27 1.27)) hide)
     )
@@
       (effects (font (size 1.27 1.27)) hide)
     )
-    (property "LCSC" "C25803" (id 4) (at 77.47 137.16 0)
+    (property "LCSC" "C269673" (id 4) (at 77.47 137.16 0)
       (effects (font (size 1.27 1.27)) hide)
     )
@@
       (effects (font (size 1.27 1.27)) hide)
     )
-    (property "LCSC" "C25803" (id 4) (at 68.58 165.1 0)
-      (effects (font (size 1.27 1.27)) hide)
-    )
+    (property "LCSC" "C269673" (id 4) (at 68.58 165.1 0)
+      (effects (font (size 1.27 1.27)) hide)
+    )

Commit message: submitted to jlcpcb
Other:
- note removed: "LCSC HAS A LOT OF DIFFERENT LCSC-NUMBERS FOR THE TLE"
- note removed: "RECONFIRM PINS ON IS3720 / IS3721 BEFORE ORDERING"
- moved on the sheet: C10, C11, C15, C16, C17, C4, C5, C6, C8, C9, J4, J5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

Commit message: error with U2
Other:
- note added: "PINS 2 AND 5 INCORRECTLY LABELED!!!"
Changed lines of the file:
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@@
     (effects (font (size 1.27 1.27)) (justify left bottom))
+  )
+  (text "PINS 2 AND 5 INCORRECTLY LABELED!!!" (at 43.18 154.305 0)
+    (effects (font (size 2.032 2.032)) (justify left bottom))
   )
   (text "Differential opamp measuring the \nvoltage across the 10 thermistor \nwith gain 1 (check...) means that \nthe rest of the board is protected \nby the 100m and 4k7 impedances. \nWill be hard to kill anything through \nthese (the resistors may die...)"
@@
   )
   (text "OPTIONAL FIT, \nDNP for full duplex on STM, \nFit for half duplex"
-    (at 100.33 102.87 180)
+    (at 100.33 102.87 0)
     (effects (font (size 1.27 1.27)) (justify right bottom))
   )

Commit message: error with U2
Parts:
- added U?: MCP6L01x-xLT, Package_TO_SOT_SMD:SOT-353_SC-70-5, symbol Amplifier_Operational:MCP6L01x-xLT
Other:
- note added: "Reduce the 470ohm resistors to 100ohm Thermister spelt wrong Repair opamp"
- note added: "Use this symbol / footprint"
Changed lines of the file:
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@@
+    (effects (font (size 1.27 1.27)) (justify left bottom))
+  )
+  (text "Reduce the 470ohm resistors to 100ohm\nThermister spelt wrong\nRepair opamp"
+    (at 97.155 170.815 0)
     (effects (font (size 1.27 1.27)) (justify left bottom))
   )
@@
   (text "Isolator decouplers\n" (at 143.51 99.06 0)
     (effects (font (size 1.27 1.27)) (justify left bottom))
+  )
+  (text "Use this symbol / footprint" (at 115.062 142.621 0)
+    (effects (font (size 2.032 2.032)) (justify left bottom))
   )
   (text "A SIDE: ISOLATED WITH ENCODER" (at 118.11 36.83 0)
@@
     (pin "2")
   )
+  (symbol (lib_id "Amplifier_Operational:MCP6L01x-xLT") (at 121.92 152.019 0) (unit 1)
+    (in_bom yes) (on_board yes) (fields_autoplaced)
+    (property "Reference" "U?" (id 0) (at 135.128 147.32 0))
+    (property "Value" "MCP6L01x-xLT" (id 1) (at 135.128 149.86 0))
+    (property "Footprint" "Package_TO_SOT_SMD:SOT-353_SC-70-5" (id 2) (at 119.38 157.099 0)
+      (effects (font (size 1.27 1.27)) (justify left) hide)
+    )
+    (property "Datasheet" "http://ww1.microchip.com/downloads/en/devicedoc/22140b.pdf" (id 3) (at 121.92 152.019 0)
+      (effects (font (size 1.27 1.27)) hide)
+    )
+    (pin "2")
+    (pin "5")
+    (pin "1")
+    (pin "3")
+    (pin "4")
+  )
   (symbol (lib_id "Connector:Conn_01x02_Male") (at 255.27 109.22 90) (unit 1)
     (in_bom no) (on_board yes)
@@
       (reference "U6") (unit 1) (value "CA-IS3721C") (footprint "Package_SO:SOIC-8_3.9x4.9mm_P1.27mm")
     )
-  )
+    (path "/71748eb4-804b-44ff-8efd-dbe46a5c4786"
+      (reference "U?") (unit 1) (value "MCP6L01x-xLT") (footprint "Package_TO_SOT_SMD:SOT-353_SC-70-5")
+    )
+  )
