File: AS5048_atmega328p/atmega328.kicad_sch (KiCad schematic)
At the start: 26 parts, among them J1 Conn_01x04, J2 Conn_01x02, J3 Conn_01x02_Male, J4 Conn_01x03, J5 Conn_01x08, J6 Conn_01x02, Q1 Si2319CDS, U1 ATmega328P-AU, U2 AS5048A, Y1 Crystal

Commit message: new notes
Other:
- note added: "Notes: Never really got this to work. decoupling caps werent doing their job on original design which could be the cause; original xtal just didnt work; this may have resulted in serial writing bad characters; and programming problems. It's not clear the clock speed would ever be fast enough for SPI communications and reasonable output"
Changed lines of the file:
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@@
     (effects (font (size 1.27 1.27)) (justify left bottom))
+  )
+  (text "Notes:\nNever really got this to work. \ndecoupling caps werent doing their job on original design which could be the cause;\noriginal xtal just didnt work;\nthis may have resulted in serial writing bad characters;\nand programming problems. \n\nIt's not clear the clock speed would ever be fast enough for\nSPI communications and reasonable output\n\n"
+    (at 87.757 124.841 0)
+    (effects (font (size 1 1)) (justify left bottom))
   )
   (global_label "SND" (shape input) (at 92.71 37.211 0) (fields_autoplaced)
